File: Node_MP3/Waggon_MP3.kicad_sch (KiCad schematic)
At the start: 85 parts, among them J1 Screw_Terminal_01x05, J10 Conn_01x01, J11 Conn_01x01, J12 Conn_01x01, J13 Conn_01x01, J14 Conn_01x01, J15 Conn_01x01, J16 Conn_01x01, J17 Conn_01x01, J18 Conn_01x01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

Commit message: Schematic of Node-MP3
Parts:
- removed C?: 100n, BBS:C_Rect_L7.0mm_W2.0mm_P5.00mm, symbol Device:C
- removed D1, D10, D11, D12, D13, D14, D15, D16, D17, D18, D2, D3, D4, D5, D6, D7, D8, D9, D?: LED, symbol Device:LED
- removed LS1: Speaker, symbol Device:Speaker
- removed R10, R11, R12, R13, R14, R15, R16, R17, R18, R19, R20, R21, R22, R23, R24, R7, R8, R9, R?: 1k5, BBS:R_7.5, symbol Device:R
- removed R25: 1k, BBS:R_7.5, symbol Device:R
- removed U?: Adafruit_MAX4466, Connector_PinHeader_2.54mm:PinHeader_1x03_P2.54mm_Vertical, symbol BBS_TGHS:Adafruit_MAX4466
- renumbered C4 to C?, C3 to C?, U2 to U?
Connections:
- net +5V: no longer names the net of A1.27 (+5V), C1.1, C2.2, C?.1, C?.1, PS1.3 (+VOUT), R1.1, R4.1, R5.1, R6.1, U1.8 (VCC), U?.1 (VCC)
- net J12: no longer names the net of U?.3 (TX)
Other:
- note added: "Controller für Waggon mit RS485"
- note removed: "D1..D6 = 2mA GN D7, D8 = 2mA GE D9 = 2mA RT"
- note removed: "Eletronic gimmick for wagon DK with mp3-player and some kind of VU-Meter. Can be controlled via I2C or RS485"
- note removed: "LED 2mA GN on Top"
- note removed: "Left side"
- note removed: "Microphone with adjustable gain"
- note removed: "Right side"
