File: Node_Rev2/Wagon.kicad_pcb (KiCad board)
At the start: 2 copper layers, 34.3 x 68.5 mm, 46 parts, among them J1 Screw_Terminal_01x05, J10 Conn_01x01, J11 Conn_01x01, J12 Conn_01x01, J13 Conn_01x01, J14 Conn_01x01, J15 Conn_01x01, J16 Conn_01x01, J17 Conn_01x01, J18 Conn_01x01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

Commit message: Test with EMQX as public broker to see, if more than one topis are possible
Other:
- net class Default removed
